Commit message: fix color warning(about a color named "2")

File: ros_urdf_learn/urdf/rbo1.urdf.xacro (robot description, xacro)
@@ -13,4 +13,7 @@
 	<color rgba="0 0 0 1"/>
 </material>
+<material name="2">
+       <color rgba="1 0 0.2 0.8"/>
+</material>
     <!-- macro -->
     <xacro:macro name="default_inertial" params="mass">
@@ -37,7 +40,5 @@
         <visual>
             <xacro:box_geometry width="${car_width}" length="${car_length}" height="${car_height}"/>
-		<material name="2">
-		     <color rgba="9 3 25 0.8"/>
-		</material>
+	    <material name="2"/>
         </visual>
         <collision>
